File: pixelD.brd (EAGLE design)
At the start: 30 parts, among them CON3 DS1066-07M-SIDE, CON4 DS1066-07M-SIDE, IC4 WS2811, IC5 LM1117-3.3-SOT223

Commit message: pixelD update
Parts:
- removed CON3, CON4: DS1066-07M-SIDE, pixel_masterlib:DS1066-08M_SIDE
- removed DRIVER1:C2, DRIVER2:C2, DRIVER3:C2: 22uF, rcl:D/7343-31R
- removed DRIVER1:D2, DRIVER2:D2, DRIVER3:D2: (no value), SparkFun-DiscreteSemi:SMA-DIODE-KIT
- removed DRIVER1:IC2, DRIVER2:IC2, DRIVER3:IC2: (no value), PT4115:PT4115
- removed DRIVER1:L2, DRIVER2:L2, DRIVER3:L2: 68uH, inductor-panasonic:ELL6
- removed DRIVER1:R2, DRIVER2:R2, DRIVER3:R2: 0.3, SparkFun-Resistors:0805
- removed LED_ANODE, LED_ANODE1, LED_ANODE2, LED_CATHODE1, LED_CATHODE2, LED_CATHODE3: WIREPADSMD5-2,5, valenok_master_library:5-2,5
- added ANODE1, ANODE2, ANODE4, CATHODE1, CATHODE2, CATHODE4: WIREPADSMD5-2,5, valenok_master_library:5-2,5
- added CON2, CON5: DS1066-07M-SIDE, pixel_masterlib:DS1066-08M_SIDE
- added D4: SMF05C, pixel_masterlib:SC70_6L
- added LED_DRV1:C2, LED_DRV2:C2, LED_DRV3:C2: 10 uF, rc:C1812
- added LED_DRV1:D1, LED_DRV2:D1, LED_DRV3:D1: CRS08-SOD123, FMU_masterlib:SOD123
- added LED_DRV1:IC4, LED_DRV2:IC4, LED_DRV3:IC4: (no value), pixel_masterlib:PT4115
- added LED_DRV1:L2, LED_DRV2:L2, LED_DRV3:L2: 47UH, power_inductors:SDR0805
- added LED_DRV1:R4, LED_DRV2:R4, LED_DRV3:R4: (no value), rc:R1206
- added R11, R12: 100R, rc:R0603
- added RN1, RN2: 510R, pixel_masterlib:CAT16-J4
- added U$6: CONNECTION, usb2can_master_lib:CONNECTION
Connections:
- removed net DRIVER1:N$1: DRIVER1:D2.A, DRIVER1:IC2.1, DRIVER1:L2.2
- removed net DRIVER2:N$1: DRIVER2:D2.A, DRIVER2:IC2.1, DRIVER2:L2.2
- removed net DRIVER3:N$1: DRIVER3:D2.A, DRIVER3:IC2.1, DRIVER3:L2.2
- removed net N$10: DRIVER2:IC2.4, DRIVER2:R2.1, LED_ANODE1.1
- removed net N$11: DRIVER2:L2.1, LED_CATHODE2.1
- removed net N$8: DRIVER3:L2.1, LED_CATHODE3.1
- removed net N$9: DRIVER1:IC2.3, IC4.1
- new net A: D4.4, R11.1
- new net B: D4.3, R12.1
- new net CLOCK: D4.6, RN1.3
- new net CLOCK_BUFFERED: RN2.2
- new net CS: D4.1, RN1.4
- new net CS_OUT: RN2.4
- new net DATA_BUFFERED: RN2.1
- new net GNDD: CON2.7, CON5.7, U$6.P$1
- new net LED_DRV1:N$2: LED_DRV1:D1.A, LED_DRV1:IC4.1, LED_DRV1:L2.1
- new net LED_DRV2:N$2: LED_DRV2:D1.A, LED_DRV2:IC4.1, LED_DRV2:L2.1
- new net LED_DRV3:N$2: LED_DRV3:D1.A, LED_DRV3:IC4.1, LED_DRV3:L2.1
- new net MOSI/DATA: D4.5, RN1.2
- new net N$12: CON2.5, RN1.6
- new net N$13: CON5.4, RN2.8
- new net N$14: CON5.6, RN2.5
- new net N$15: CON5.5, RN2.7
- new net N$16: CON2.6, RN1.5
- new net N$17: CATHODE4.1, LED_DRV3:L2.2
- new net N$18: ANODE4.1, LED_DRV3:IC4.4, LED_DRV3:R4.P$1
- new net N$6: CON2.4, RN1.7
- new net PWM1: IC4.1, LED_DRV3:IC4.3
- new net PWM2: IC4.2, LED_DRV1:IC4.3
- new net RS485_A1: CON2.2, CON5.2, R12.2
- new net RS485_B1: CON2.3, CON5.3, R11.2
- net GND: now also D4.2, LED_DRV1:C2.P$1, LED_DRV1:IC4.2, LED_DRV1:IC4.2A, LED_DRV2:C2.P$1, LED_DRV2:IC4.2, LED_DRV2:IC4.2A, LED_DRV3:C2.P$1, LED_DRV3:IC4.2, LED_DRV3:IC4.2A, U$6.P$2; no longer CON3.7, CON4.7, DRIVER1:C2.-, DRIVER1:IC2.2, DRIVER1:IC2.2A, DRIVER2:C2.-, DRIVER2:IC2.2, DRIVER2:IC2.2A, DRIVER3:C2.-, DRIVER3:IC2.2, DRIVER3:IC2.2A
- net N$2: now also CATHODE1.1, LED_DRV1:L2.2; no longer DRIVER2:IC2.3, IC4.2
- net N$4: now also ANODE1.1, LED_DRV1:IC4.4, LED_DRV1:R4.P$1; no longer DRIVER1:IC2.4, DRIVER1:R2.1, LED_ANODE.1
- net N$5: now also CATHODE2.1, LED_DRV2:L2.2; no longer DRIVER1:L2.1, LED_CATHODE1.1
- net N$7: now also ANODE2.1, LED_DRV2:IC4.4, LED_DRV2:R4.P$1; no longer DRIVER3:IC2.4, DRIVER3:R2.1, LED_ANODE2.1
- net PWM_B: now also LED_DRV2:IC4.3; no longer DRIVER3:IC2.3
- net VDD_12V: no longer DRIVER1:C2.+, DRIVER1:D2.C, DRIVER1:IC2.5, DRIVER1:R2.2, DRIVER2:C2.+, DRIVER2:D2.C, DRIVER2:IC2.5, DRIVER2:R2.2, DRIVER3:C2.+, DRIVER3:D2.C, DRIVER3:IC2.5, DRIVER3:R2.2
- net VDD_24V: now also CON2.1, CON5.1, LED_DRV1:C2.P$2, LED_DRV1:D1.C, LED_DRV1:IC4.5, LED_DRV1:R4.P$2, LED_DRV2:C2.P$2, LED_DRV2:D1.C, LED_DRV2:IC4.5, LED_DRV2:R4.P$2, LED_DRV3:C2.P$2, LED_DRV3:D1.C, LED_DRV3:IC4.5, LED_DRV3:R4.P$2; no longer CON3.1, CON4.1
