File: pixelD.sch (EAGLE design)
At the start: 15 parts, among them CON3 DS1066-07M-SIDE, CON4 DS1066-07M-SIDE, IC4 WS2811, IC5 LM1117-3.3-SOT223

Commit message: pixelD update
Parts:
- removed CON3, CON4: DS1066-07M-SIDE, pixel_masterlib:DS1066-07M-SIDE
- removed LED_ANODE, LED_ANODE1, LED_ANODE2, LED_CATHODE1, LED_CATHODE2, LED_CATHODE3: WIREPADSMD5-2,5, valenok_master_library:WIREPADSMD5-2,5
- added ANODE1, ANODE2, ANODE4, CATHODE1, CATHODE2, CATHODE4: WIREPADSMD5-2,5, valenok_master_library:WIREPADSMD5-2,5
- added CON2, CON5: DS1066-07M-SIDE, pixel_masterlib:DS1066-07M-SIDE
- added D4: SMF05C, pixel_masterlib:SMF05C
- added R11, R12: 100R, rc:R-0603
- added RN1, RN2: 510R, pixel_masterlib:RESISTOR_ARRAY
- added U$6: CONNECTION, usb2can_master_lib:CONNECTION
Connections:
- net N$2 renamed PWM2
- net N$9 renamed PWM1
- removed net N$10: LED_ANODE1.P
- removed net N$11: LED_CATHODE2.P
- removed net N$8: LED_CATHODE3.P
- new net A: D4.D3, R11.1
- new net ANODE: IC4.CSN, R4.1
- new net B: D4.D2, R12.1
- new net CLOCK: D4.D5, RN1.3
- new net CLOCK_BUFFERED: RN2.2
- new net CS: D4.D1, RN1.4
- new net CS_OUT: RN2.4
- new net DATA_BUFFERED: RN2.1
- new net DIM: IC4.DIM
- new net GNDD: CON2.7, CON5.7, U$6.P$1
- new net MOSI/DATA: D4.D4, RN1.2
- new net N$12: CON2.5, RN1.6
- new net N$13: CON5.4, RN2.8
- new net N$14: CON5.6, RN2.5
- new net N$15: CON5.5, RN2.7
- new net N$16: CON2.6, RN1.5
- new net N$17: CATHODE4.P
- new net N$18: ANODE4.P
- new net N$2: CATHODE1.P, IC4.SW
- new net N$6: CON2.4, RN1.7
- new net RS485_A1: CON2.2, CON5.2, R12.2
- new net RS485_B1: CON2.3, CON5.3, R11.2
- new net SUPPLY: IC4.VIN, R4.2
- net GND: now also D4.G, U$6.P$2; no longer CON3.7, CON4.7
- net N$4: now also ANODE1.P; no longer LED_ANODE.P
- net N$5: now also CATHODE2.P; no longer LED_CATHODE1.P
- net N$7: now also ANODE2.P; no longer LED_ANODE2.P
- net VDD_24V: now also CON2.1, CON5.1; no longer CON3.1, CON4.1
Other:
- moved on the sheet: C4, C5, C6, IC4, IC5, R4, R6
