File: pixel8.brd (EAGLE design)
At the start: 18 parts, among them CON3 DS1066-07M-SIDE, CON4 DS1066-07M-SIDE

Commit message: pixel8 update
Parts:
- removed CON4: DS1066-07M-SIDE, pixel_masterlib:DS1066-08M_SIDE
- removed D1, D2, D3: (no value), SparkFun-DiscreteSemi:SMA-DIODE-KIT
- removed IC1, IC2, IC3: (no value), PT4115:PT4115
- removed L1, L2, L3: 68uH, inductor-panasonic:ELL6
- removed R3: 0.3, SparkFun-Resistors:0805
- added ANODE1, ANODE2, ANODE3, CATHODE1, CATHODE2, CATHODE3: WIREPADSMD5-2,5, valenok_master_library:5-2,5
- added C19, C20: (no value), rc:C0603
- added C26: 100 nF, rc:C0603
- added CON1, CON2: DS1066-07M-SIDE, pixel_masterlib:DS1066-08M_SIDE
- added D4: SMF05C, pixel_masterlib:SC70_6L
- added IC4: ST3485SOIC8, pixel_masterlib:SOIC8
- added IC6, IC7: MC74VHC1GT125, pixel_masterlib:SOT23-5
- added LED_DRV1:C1, LED_DRV2:C1, LED_DRV3:C1: 10 uF, rc:C1812
- added LED_DRV1:D1, LED_DRV2:D1, LED_DRV3:D1: CRS08-SOD123, FMU_masterlib:SOD123
- added LED_DRV1:IC1, LED_DRV2:IC1, LED_DRV3:IC1: (no value), pixel_masterlib:PT4115
- added LED_DRV1:L1, LED_DRV2:L1, LED_DRV3:L1: 47UH, power_inductors:SDR0805
- added LED_DRV1:R1, LED_DRV2:R1, LED_DRV3:R1: (no value), rc:R1206
- added R5: 120R, rc:R0603
- added R8: 10K, rc:R0603
- added RN1, RN2: 510R, pixel_masterlib:CAT16-J4
- added SJ2: (no value), eth_conv_master_lib:RES_0
- added U$1: (no value), pixel_masterlib:PIXEL8_BOARD_OUTLINE
- added U$2, U$3, U$4, U$5: (no value), pixel_masterlib:MOUNTING_HOLE_M3
- added U$6: CONNECTION, usb2can_master_lib:CONNECTION
- added Z1: 16MHz, watchdog_master_library:OSCILLATOR-3.2X2.5
- C1: value 22uF -> 0.1uF; device rcl:D/7343-31R -> rc:C0603
- C2, C3: value 22uF -> 100 nF; device rcl:D/7343-31R -> rc:C0603
- CON3: value DS1066-07M-SIDE -> PINHEAD_1X02-2.54; device pixel_masterlib:DS1066-08M_SIDE -> pinhead:1X02-PTH-2.54
- R1, R2: value 0.3 -> 100R; device SparkFun-Resistors:0805 -> rc:R0603
- moved R1 98.7 mm to (-11.1, 18.6), turned to 180 degrees
- moved R2 98.2 mm to (-11.1, 17.4), turned to 180 degrees
- moved C2 95.5 mm to (4.85, 14.6)
- moved C1 91.1 mm to (-4.35, 15.5), turned to 180 degrees
- moved C3 88.2 mm to (1.85, 8.20), turned to 90 degrees
- moved MODULE1 37.6 mm to (0.00, 7.55)
- moved CON3 11.9 mm to (17.4, -11.8), turned to 270 degrees
Connections:
- removed net B+: IC3.4, R3.1
- removed net B-: L3.1
- removed net G+: IC2.4, R2.1
- removed net G-: L2.1
- removed net N$14: CON3.4
- removed net N$16: CON3.5
- removed net N$18: CON3.6
- removed net N$19: CON4.4
- removed net N$20: CON4.5
- removed net N$21: CON4.6
- removed net PWM_B: IC3.3
- removed net PWM_G: IC2.3
- removed net PWM_R: IC1.3
- removed net R+: IC1.4, R1.1
- removed net R-: L1.1
- removed net RS485_A: CON3.2, CON4.2
- removed net RS485_B: CON3.3, CON4.3
- removed net VCC: C1.+, C2.+, C3.+, D1.C, D2.C, D3.C, IC1.5, IC2.5, IC3.5, R1.2, R2.2, R3.2
- removed net VDD_24V: CON3.1, CON4.1
- new net A: D4.4, IC4.6, R2.1, R5.2
- new net B: D4.3, IC4.7, R1.1, SJ2.1
- new net CLOCK: D4.6, IC6.2, MODULE1.15, RN1.3
- new net CLOCK_BUFFERED: IC6.4, RN2.2
- new net CS: D4.1, MODULE1.10, RN1.4
- new net CS_OUT: MODULE1.13, RN2.4
- new net DATA_BUFFERED: IC7.4, RN2.1
- new net GNDD: CON1.7, CON2.7, U$6.P$1
- new net LED_DRV1:N$2: LED_DRV1:D1.A, LED_DRV1:IC1.1, LED_DRV1:L1.1
- new net LED_DRV2:N$2: LED_DRV2:D1.A, LED_DRV2:IC1.1, LED_DRV2:L1.1
- new net LED_DRV3:N$2: LED_DRV3:D1.A, LED_DRV3:IC1.1, LED_DRV3:L1.1
- new net MISO: MODULE1.17
- new net MOSI/DATA: D4.5, IC7.2, MODULE1.16, RN1.2
- new net N$1: CON2.4, RN2.8
- new net N$10: ANODE1.1, LED_DRV1:IC1.4, LED_DRV1:R1.P$1
- new net N$11: CON1.4, RN1.7
- new net N$12: CON1.5, RN1.6
- new net N$13: CON1.6, RN1.5
- new net N$15: CON2.5, RN2.7
- new net N$17: ANODE3.1, LED_DRV3:IC1.4, LED_DRV3:R1.P$1
- new net N$3: CON2.6, RN2.5
- new net N$5: R5.1, SJ2.2
- new net N$6: C19.1, MODULE1.5, Z1.1
- new net N$8: CATHODE1.1, LED_DRV1:L1.2
- new net N$9: C20.1, MODULE1.6, Z1.3
- new net PWM1: LED_DRV1:IC1.3, MODULE1.1
- new net PWM2: LED_DRV2:IC1.3, MODULE1.20
- new net PWM3: LED_DRV3:IC1.3, MODULE1.19
- new net RE/DE: IC4.2, IC4.3, MODULE1.3
- new net RS485_A1: CON1.2, CON2.2, R1.2
- new net RS485_B1: CON1.3, CON2.3, R2.2
- new net RX/TX: IC4.1, IC4.4, MODULE1.2
- new net SWIM: MODULE1.18
- new net TEMP: C26.2, CON3.1, MODULE1.14, R8.2
- new net VDD_12V: CON1.1, CON2.1, LED_DRV1:C1.P$2, LED_DRV1:D1.C, LED_DRV1:IC1.5, LED_DRV1:R1.P$2, LED_DRV2:C1.P$2, LED_DRV2:D1.C, LED_DRV2:IC1.5, LED_DRV2:R1.P$2, LED_DRV3:C1.P$2, LED_DRV3:D1.C, LED_DRV3:IC1.5, LED_DRV3:R1.P$2
- new net VDD_3V3: C1.2, C2.2, C3.2, CON3.2, IC4.8, IC6.5, IC7.5, MODULE1.9
- net GND: now also C1.1, C19.2, C2.1, C20.2, C26.1, C3.1, D4.2, IC4.5, IC6.3, IC7.3, LED_DRV1:C1.P$1, LED_DRV1:IC1.2, LED_DRV1:IC1.2A, LED_DRV2:C1.P$1, LED_DRV2:IC1.2, LED_DRV2:IC1.2A, LED_DRV3:C1.P$1, LED_DRV3:IC1.2, LED_DRV3:IC1.2A, MODULE1.7, R8.1, U$6.P$2, Z1.2, Z1.4; no longer C1.-, C2.-, C3.-, CON3.7, CON4.7, IC1.2, IC1.2A, IC2.2, IC2.2A, IC3.2, IC3.2A
- net N$2: now also CATHODE2.1, LED_DRV2:L1.2; no longer D1.A, IC1.1, L1.2
- net N$4: now also ANODE2.1, LED_DRV2:IC1.4, LED_DRV2:R1.P$1; no longer D2.A, IC2.1, L2.2
- net N$7: now also CATHODE3.1, LED_DRV3:L1.2; no longer D3.A, IC3.1, L3.2
Routing:
- net B: track 0.00 -> 14.0 mm
- net A: track 0.00 -> 8.38 mm
- net N$9: track 0.00 -> 4.81 mm
- net N$6: track 0.00 -> 1.97 mm
- net N$5: track 0.00 -> 1.83 mm
- added copper zone on layer 16, net GND
Other:
- board outline added: 39.5 x 46 mm

Commit message: pixel8 update
Parts:
- removed C19, C20: (no value), rc:C0603
- removed C26: 100 nF, rc:C0603
- removed LED_DRV1:C1, LED_DRV2:C1, LED_DRV3:C1: 10 uF, rc:C1812
- removed LED_DRV1:D1, LED_DRV2:D1, LED_DRV3:D1: CRS08-SOD123, FMU_masterlib:SOD123
- removed LED_DRV1:IC1, LED_DRV2:IC1, LED_DRV3:IC1: (no value), pixel_masterlib:PT4115
- removed LED_DRV1:L1, LED_DRV2:L1, LED_DRV3:L1: 47UH, power_inductors:SDR0805
- removed LED_DRV1:R1, LED_DRV2:R1, LED_DRV3:R1: (no value), rc:R1206
- removed R8: 10K, rc:R0603
- added C101, C201, C301: 10 uF, rc:C1812
- added C4, C5: (no value), rc:C0603
- added C6: 100 nF, rc:C0603
- added D101, D201, D301: CRS08-SOD123, FMU_masterlib:SOD123
- added IC101, IC201, IC301: (no value), pixel_masterlib:PT4115
- added L101, L201, L301: 47UH, power_inductors:SDR0805
- added R101, R201, R301: (no value), rc:R1206
- added R3: 10K, rc:R0603
- moved CON3 9.06 mm to (11.2, -5.20)
- moved ANODE3 8.33 mm to (10.6, -19.9)
- moved ANODE2 5.18 mm to (2.12, -19.9)
- moved CATHODE3 4.73 mm to (6.38, -19.9)
- moved CATHODE1 4.40 mm to (-6.38, -19.9)
- moved ANODE1 4.05 mm to (-10.6, -19.9)
- moved D4 1.99 mm to (-0.47, 9.15), turned to 90 degrees
- moved C1 1.07 mm to (-4.55, 16.6)
- moved U$6 0.87 mm to (-11.3, 1.10)
- moved RN1 0.84 mm to (-4.35, 11.6)
- moved C3 0.67 mm to (1.35, 8.65), turned to 270 degrees
- moved Z1 0.55 mm to (-4.30, 6.30)
- moved IC4 0.50 mm to (-2.35, 20.1)
- moved RN2 0.20 mm to (4.50, 5.25)
- moved CATHODE2 0.06 mm to (-2.12, -19.9)
Connections:
- net RS485_A1 renamed RS485_A
- net RS485_B1 renamed RS485_B
- removed net LED_DRV1:N$2: LED_DRV1:D1.A, LED_DRV1:IC1.1, LED_DRV1:L1.1
- removed net LED_DRV2:N$2: LED_DRV2:D1.A, LED_DRV2:IC1.1, LED_DRV2:L1.1
- removed net LED_DRV3:N$2: LED_DRV3:D1.A, LED_DRV3:IC1.1, LED_DRV3:L1.1
- removed net N$10: ANODE1.1, LED_DRV1:IC1.4, LED_DRV1:R1.P$1
- removed net N$17: ANODE3.1, LED_DRV3:IC1.4, LED_DRV3:R1.P$1
- removed net N$2: CATHODE2.1, LED_DRV2:L1.2
- removed net N$4: ANODE2.1, LED_DRV2:IC1.4, LED_DRV2:R1.P$1
- removed net N$7: CATHODE3.1, LED_DRV3:L1.2
- removed net N$8: CATHODE1.1, LED_DRV1:L1.2
- new net A1: ANODE1.1, IC101.4, R101.P$1
- new net A2: ANODE2.1, IC201.4, R201.P$1
- new net A3: ANODE3.1, IC301.4, R301.P$1
- new net C1: CATHODE1.1, L101.2
- new net C2: CATHODE2.1, L201.2
- new net C3: CATHODE3.1, L301.2
- new net LED_DRV1:SW: D101.A, IC101.1, L101.1
- new net LED_DRV2:SW: D201.A, IC201.1, L201.1
- new net LED_DRV3:SW: D301.A, IC301.1, L301.1
- net GND: now also C101.P$1, C201.P$1, C301.P$1, C4.2, C5.2, C6.1, IC101.2, IC101.2A, IC201.2, IC201.2A, IC301.2, IC301.2A, R3.1; no longer C19.2, C20.2, C26.1, LED_DRV1:C1.P$1, LED_DRV1:IC1.2, LED_DRV1:IC1.2A, LED_DRV2:C1.P$1, LED_DRV2:IC1.2, LED_DRV2:IC1.2A, LED_DRV3:C1.P$1, LED_DRV3:IC1.2, LED_DRV3:IC1.2A, R8.1
- net N$6: now also C4.1; no longer C19.1
- net N$9: now also C5.1; no longer C20.1
- net PWM1: now also IC101.3; no longer LED_DRV1:IC1.3
- net PWM2: now also IC201.3; no longer LED_DRV2:IC1.3
- net PWM3: now also IC301.3; no longer LED_DRV3:IC1.3
- net TEMP: now also C6.2, R3.2; no longer C26.2, R8.2
- net VDD_12V: now also C101.P$2, C201.P$2, C301.P$2, D101.C, D201.C, D301.C, IC101.5, IC201.5, IC301.5, R101.P$2, R201.P$2, R301.P$2; no longer LED_DRV1:C1.P$2, LED_DRV1:D1.C, LED_DRV1:IC1.5, LED_DRV1:R1.P$2, LED_DRV2:C1.P$2, LED_DRV2:D1.C, LED_DRV2:IC1.5, LED_DRV2:R1.P$2, LED_DRV3:C1.P$2, LED_DRV3:D1.C, LED_DRV3:IC1.5, LED_DRV3:R1.P$2
Routing:
- net VDD_12V: track 0.00 -> 34.3 mm, vias 0 -> 12
- net A1: track 0.00 -> 19.9 mm, vias 0 -> 12
- net GND: track 0.00 -> 18.9 mm, vias 0 -> 33
- net RE/DE: track 0.00 -> 16.7 mm
- net A2: track 0.00 -> 15.5 mm, vias 0 -> 12
- net RX/TX: track 0.00 -> 14.5 mm
- net A3: track 0.00 -> 11.3 mm, vias 0 -> 12
- net TEMP: track 0.00 -> 8.33 mm
- net N$11: track 0.00 -> 8.08 mm
- net PWM2: track 0.00 -> 7.65 mm
- net N$12: track 0.00 -> 7.10 mm
- net CS_OUT: track 0.00 -> 6.68 mm
- net N$13: track 0.00 -> 6.61 mm
- net N$1: track 0.00 -> 6.41 mm
- net N$15: track 0.00 -> 6.24 mm
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- added copper zone on layer 1, net A1
- added copper zone on layer 16, net A1
- added copper zone on layer 1, net A2
- added copper zone on layer 16, net A2
- added copper zone on layer 1, net A3
- added copper zone on layer 16, net A3
- added copper zone on layer 1, net C1
- added copper zone on layer 1, net C2
- added copper zone on layer 1, net C3
- added copper zone on layer 1, net GND
- added copper zone on layer 1, net LED_DRV1:SW
- added copper zone on layer 1, net LED_DRV2:SW
- added copper zone on layer 1, net LED_DRV3:SW
- added copper zone on layer 1, net VDD_12V
- added copper zone on layer 16, net VDD_12V
