File: pixel32.sch (EAGLE design)
At the start: 49 parts, among them CON1 DS1066-07M-SIDE, CON2 DS1066-07M-SIDE, CON3 PINHEAD_1X02-2.54, CON4 PINHEAD_1X03-2.54, IC1 STM32F030K6TX-LQFP32(7X7), IC3 ST3485SOIC8, IC6 MC74VHC1GT125, IC7 MC74VHC1GT125, IC8 LM317

Commit message: Routing
Parts:
- IC8: device masterlib:LM317 -> pixel_masterlib:LM317
- LED_ANODE, LED_CATHODE1, LED_CATHODE2, LED_CATHODE3: device valenok_master_library:WIREPADSMD5-2,5 -> wirepad:WIREPADSMD5-2,5
- MODULE1: device ali_modules:GW1584 -> pixel_masterlib:GW1584
- SJ1, SJ2, SJ3: device eth_conv_master_lib:SOLDER_JOINT -> misc:SOLDER_JOINT
- Z1: device watchdog_master_library:CRYSTAL-3.2X2.5-4P -> crystals:CRYSTAL-3.2X2.5-4P
Connections:
- net A: now also D1.D3; no longer D1.D2
- net B: now also D1.D2; no longer D1.D3
Changed lines of the file:
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@@
 <part name="R1" library="rc" deviceset="R" device="-0603" value="22R"/>
 <part name="R2" library="rc" deviceset="R" device="-R1206" value="2R"/>
-<part name="D1" library="FMU_masterlib" deviceset="CRS08" device="-SOD123"/>
+<part name="D1" library="pixel_masterlib" deviceset="CRS08" device="-SOD123"/>
 <part name="IC1" library="pixel_masterlib" deviceset="IRS44273L" device=""/>
 <part name="C2" library="rc" deviceset="C" device="-0805" value="1 uF"/>
@@
 <part name="C3" library="rc" deviceset="C" device="-0603" value="100 nF"/>
 <part name="GND1" library="supply_symbols" deviceset="GND" device="" value="GND"/>
-<part name="TP1" library="pixhawk2" deviceset="PAD" device=".05">
+<part name="TP1" library="misc" deviceset="PAD" device=".05">
 <attribute name="BOM" value="EXCLUDE"/>
 <attribute name="PARTNO" value="*"/>
 </part>
-<part name="TP2" library="pixhawk2" deviceset="PAD" device=".05">
+<part name="TP2" library="misc" deviceset="PAD" device=".05">
 <attribute name="BOM" value="EXCLUDE"/>
 <attribute name="PARTNO" value="*"/>
 </part>
-<part name="TP3" library="pixhawk2" deviceset="PAD" device=".05">
+<part name="TP3" library="misc" deviceset="PAD" device=".05">
 <attribute name="BOM" value="EXCLUDE"/>
 <attribute name="PARTNO" value="*"/>
@@
 </modules>
 <parts>
-<part name="MODULE1" library="ali_modules" deviceset="GW1584" device=""/>
+<part name="MODULE1" library="pixel_masterlib" deviceset="GW1584" device=""/>
 <part name="GND24" library="supply_symbols" deviceset="GND" device="" value="GND"/>
 <part name="GND25" library="supply_symbols" deviceset="GND" device="" value="GND"/>
@@
 <part name="GND20" library="supply_symbols" deviceset="GND" device="" value="GND"/>
 <part name="GND21" library="supply_symbols" deviceset="GND" device="" value="GND"/>
-<part name="Z1" library="watchdog_master_library" deviceset="CRYSTAL" device="-3.2X2.5-4P" value="16MHz"/>
+<part name="Z1" library="crystals" deviceset="CRYSTAL" device="-3.2X2.5-4P" value="16MHz"/>
 <part name="+P7" library="supply_symbols" deviceset="24V" device=""/>
 <part name="CON1" library="pixel_masterlib" deviceset="DS1066-07M" device="-SIDE"/>
@@
 <part name="GND29" library="supply_symbols" deviceset="GND" device="" value="GND"/>
 <part name="+P10" library="supply_symbols" deviceset="3.3V" device=""/>
-<part name="SJ2" library="eth_conv_master_lib" deviceset="SOLDER_JOINT" device=""/>
+<part name="SJ2" library="misc" deviceset="SOLDER_JOINT" device=""/>
 <part name="RN1" library="pixel_masterlib" deviceset="RESISTOR_ARRAY" device="" value="510R">
 <attribute name="DIGIKEY#" value="CAT16-511J4LF-ND"/>
@@
 <part name="+P3" library="supply_symbols" deviceset="24V" device=""/>
 <part name="+P1" library="supply_symbols" deviceset="12V" device=""/>
-<part name="LED_CATHODE1" library="valenok_master_library" deviceset="WIREPAD" device="SMD5-2,5"/>
-<part name="LED_CATHODE2" library="valenok_master_library" deviceset="WIREPAD" device="SMD5-2,5"/>
-<part name="LED_CATHODE3" library="valenok_master_library" deviceset="WIREPAD" device="SMD5-2,5"/>
-<part name="LED_ANODE" library="valenok_master_library" deviceset="WIREPAD" device="SMD5-2,5"/>
+<part name="LED_CATHODE1" library="wirepad" deviceset="WIREPAD" device="SMD5-2,5"/>
+<part name="LED_CATHODE2" library="wirepad" deviceset="WIREPAD" device="SMD5-2,5"/>
+<part name="LED_CATHODE3" library="wirepad" deviceset="WIREPAD" device="SMD5-2,5"/>
+<part name="LED_ANODE" library="wirepad" deviceset="WIREPAD" device="SMD5-2,5"/>
 <part name="R8" library="rc" deviceset="R" device="-0603" value="10K"/>
 <part name="CON3" library="pinhead" deviceset="PINHEAD_1X02" device="-2.54"/>
@@
 <part name="GND38" library="supply_symbols" deviceset="GND" device="" value="GND"/>
 <part name="+P11" library="supply_symbols" deviceset="12V" device=""/>
-<part name="IC8" library="masterlib" deviceset="LM317" device=""/>
+<part name="IC8" library="pixel_masterlib" deviceset="LM317" device=""/>
 <part name="R6" library="rc" deviceset="R" device="-0805" value="1K"/>
 <part name="R7" library="rc" deviceset="R" device="-0805" value="5K6"/>
@@
 <part name="GND22" library="supply_symbols" deviceset="GNDD" device="" value="GNDD"/>
 <part name="GND23" library="supply_symbols" deviceset="GNDD" device="" value="GNDD"/>
-<part name="SJ1" library="eth_conv_master_lib" deviceset="SOLDER_JOINT" device=""/>
+<part name="SJ1" library="misc" deviceset="SOLDER_JOINT" device=""/>
 <part name="+P2" library="supply_symbols" deviceset="3.3V" device=""/>
-<part name="SJ3" library="eth_conv_master_lib" deviceset="SOLDER_JOINT" device=""/>
+<part name="SJ3" library="misc" deviceset="SOLDER_JOINT" device=""/>
 <part name="+P4" library="supply_symbols" deviceset="12V" device=""/>
 <part name="+P14" library="supply_symbols" deviceset="24V" device=""/>
@@
 <segment>
 <pinref part="R12" gate="G$1" pin="1"/>
-<wire x1="317.5" y1="241.3" x2="304.8" y2="241.3" width="0.1524" layer="91"/>
 <label x="292.1" y="241.3" size="1.27" layer="95" rot="R180" xref="yes"/>
-<pinref part="D1" gate="G$1" pin="D3"/>
-<wire x1="304.8" y1="241.3" x2="292.1" y2="241.3" width="0.1524" layer="91"/>
-<wire x1="304.8" y1="223.52" x2="304.8" y2="241.3" width="0.1524" layer="91"/>
-<junction x="304.8" y="241.3"/>
+<wire x1="317.5" y1="241.3" x2="309.88" y2="241.3" width="0.1524" layer="91"/>
+<pinref part="D1" gate="G$1" pin="D2"/>
+<wire x1="309.88" y1="241.3" x2="292.1" y2="241.3" width="0.1524" layer="91"/>
+<wire x1="304.8" y1="208.28" x2="304.8" y2="205.74" width="0.1524" layer="91"/>
+<wire x1="304.8" y1="205.74" x2="309.88" y2="205.74" width="0.1524" layer="91"/>
+<wire x1="309.88" y1="205.74" x2="309.88" y2="241.3" width="0.1524" layer="91"/>
+<junction x="309.88" y="241.3"/>
 </segment>
 </net>
@@
 <segment>
 <pinref part="R11" gate="G$1" pin="1"/>
-<wire x1="317.5" y1="238.76" x2="309.88" y2="238.76" width="0.1524" layer="91"/>
 <label x="292.1" y="238.76" size="1.27" layer="95" rot="R180" xref="yes"/>
-<pinref part="D1" gate="G$1" pin="D2"/>
-<wire x1="309.88" y1="238.76" x2="292.1" y2="238.76" width="0.1524" layer="91"/>
-<wire x1="304.8" y1="208.28" x2="304.8" y2="205.74" width="0.1524" layer="91"/>
-<wire x1="304.8" y1="205.74" x2="309.88" y2="205.74" width="0.1524" layer="91"/>
-<wire x1="309.88" y1="205.74" x2="309.88" y2="238.76" width="0.1524" layer="91"/>
-<junction x="309.88" y="238.76"/>
-</segment>
-</net>
+<wire x1="317.5" y1="238.76" x2="304.8" y2="238.76" width="0.1524" layer="91"/>
+<pinref part="D1" gate="G$1" pin="D3"/>
+<wire x1="304.8" y1="238.76" x2="292.1" y2="238.76" width="0.1524" layer="91"/>
+<wire x1="304.8" y1="223.52" x2="304.8" y2="238.76" width="0.1524" layer="91"/>
+<junction x="304.8" y="238.76"/>
+</segment>
+</net>

Commit message: Routing
Connections:
- removed net N$15: CON2.5, RN2.7
- new net N$7: CON2.5, RN2.6
- net CLOCK_BUFFERED: now also RN2.4; no longer RN2.2
- net CS_OUT: now also RN2.1; no longer RN2.4
- net DATA_BUFFERED: now also RN2.3; no longer RN2.1
- net LED1_CURRENT: now also IC1.PA7/C1N; no longer IC1.PA4
- net LED2_CURRENT: now also IC1.PB0/C2N; no longer IC1.PA5
- net LED3_CURRENT: now also IC1.PB1/C3N; no longer IC1.PA6
- net TEMP: now also IC1.PA4; no longer IC1.PB0/C2N
Other:
- moved on the sheet: RN2
Changed lines of the file:
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@@
 <instance part="SJ2" gate="G$1" x="266.7" y="99.06" rot="R270"/>
 <instance part="RN1" gate="G$1" x="317.5" y="223.52"/>
-<instance part="RN2" gate="G$1" x="317.5" y="175.26"/>
+<instance part="RN2" gate="G$1" x="312.42" y="177.8"/>
 <instance part="IC6" gate="G$1" x="241.3" y="172.72"/>
 <instance part="IC7" gate="G$1" x="241.3" y="149.86"/>
@@
 <net name="LED1_CURRENT" class="0">
 <segment>
-<pinref part="IC1" gate="IC" pin="PA4"/>
-<wire x1="78.74" y1="185.42" x2="78.74" y2="182.88" width="0.1524" layer="91"/>
-<label x="78.74" y="182.88" size="1.27" layer="95" font="vector" rot="R270" xref="yes"/>
+<label x="86.36" y="172.72" size="1.27" layer="95" font="vector" rot="R270" xref="yes"/>
+<pinref part="IC1" gate="IC" pin="PA7/C1N"/>
+<wire x1="86.36" y1="172.72" x2="86.36" y2="185.42" width="0.1524" layer="91"/>
 </segment>
 <segment>
@@
 <net name="LED2_CURRENT" class="0">
 <segment>
-<pinref part="IC1" gate="IC" pin="PA5"/>
-<wire x1="81.28" y1="185.42" x2="81.28" y2="182.88" width="0.1524" layer="91"/>
-<label x="81.28" y="182.88" size="1.27" layer="95" font="vector" rot="MR270" xref="yes"/>
+<label x="88.9" y="172.72" size="1.27" layer="95" font="vector" rot="MR270" xref="yes"/>
+<pinref part="IC1" gate="IC" pin="PB0/C2N"/>
+<wire x1="88.9" y1="172.72" x2="88.9" y2="185.42" width="0.1524" layer="91"/>
 </segment>
 <segment>
@@
 <net name="LED3_CURRENT" class="0">
 <segment>
-<pinref part="IC1" gate="IC" pin="PA6"/>
-<wire x1="83.82" y1="185.42" x2="83.82" y2="182.88" width="0.1524" layer="91"/>
-<label x="83.82" y="182.88" size="1.27" layer="95" font="vector" rot="MR270" xref="yes"/>
+<wire x1="91.44" y1="185.42" x2="91.44" y2="172.72" width="0.1524" layer="91"/>
+<label x="91.44" y="172.72" size="1.27" layer="95" font="vector" rot="MR270" xref="yes"/>
+<pinref part="IC1" gate="IC" pin="PB1/C3N"/>
 </segment>
 <segment>
@@
 <net name="TEMP" class="0">
 <segment>
-<pinref part="IC1" gate="IC" pin="PB0/C2N"/>
-<wire x1="88.9" y1="185.42" x2="88.9" y2="182.88" width="0.1524" layer="91"/>
-<label x="88.9" y="182.88" size="1.27" layer="95" font="vector" rot="MR270" xref="yes"/>
+<label x="78.74" y="180.34" size="1.27" layer="95" font="vector" rot="MR270" xref="yes"/>
+<pinref part="IC1" gate="IC" pin="PA4"/>
+<wire x1="78.74" y1="180.34" x2="78.74" y2="185.42" width="0.1524" layer="91"/>
 </segment>
 <segment>
@@
 <net name="RS485_B" class="0">
 <segment>
-<pinref part="CON2" gate="G$1" pin="3"/>
-<wire x1="340.36" y1="187.96" x2="330.2" y2="187.96" width="0.1524" layer="91"/>
+<pinref part="CON1" gate="G$1" pin="3"/>
 <wire x1="330.2" y1="187.96" x2="330.2" y2="233.68" width="0.1524" layer="91"/>
-<pinref part="CON1" gate="G$1" pin="3"/>
 <wire x1="330.2" y1="233.68" x2="368.3" y2="233.68" width="0.1524" layer="91"/>
 <junction x="330.2" y="233.68"/>
@@
 <pinref part="R11" gate="G$1" pin="2"/>
 <wire x1="330.2" y1="238.76" x2="327.66" y2="238.76" width="0.1524" layer="91"/>
+<pinref part="CON2" gate="G$1" pin="3"/>
+<wire x1="340.36" y1="187.96" x2="330.2" y2="187.96" width="0.1524" layer="91"/>
 </segment>
 </net>
 <net name="RS485_A" class="0">
 <segment>
-<pinref part="CON2" gate="G$1" pin="2"/>
-<wire x1="340.36" y1="190.5" x2="332.74" y2="190.5" width="0.1524" layer="91"/>
+<pinref part="CON1" gate="G$1" pin="2"/>
 <wire x1="332.74" y1="190.5" x2="332.74" y2="236.22" width="0.1524" layer="91"/>
-<pinref part="CON1" gate="G$1" pin="2"/>
 <wire x1="332.74" y1="236.22" x2="368.3" y2="236.22" width="0.1524" layer="91"/>
 <wire x1="332.74" y1="236.22" x2="332.74" y2="241.3" width="0.1524" layer="91"/>
@@
 <pinref part="R12" gate="G$1" pin="2"/>
 <wire x1="332.74" y1="241.3" x2="327.66" y2="241.3" width="0.1524" layer="91"/>
+<pinref part="CON2" gate="G$1" pin="2"/>
+<wire x1="340.36" y1="190.5" x2="332.74" y2="190.5" width="0.1524" layer="91"/>
 </segment>
 </net>
@@
 <pinref part="RN1" gate="G$1" pin="6"/>
 <wire x1="327.66" y1="228.6" x2="368.3" y2="228.6" width="0.1524" layer="91"/>
-</segment>
-</net>
-<net name="N$14" class="0">
-<segment>
-<pinref part="CON2" gate="G$1" pin="4"/>
-<wire x1="327.66" y1="185.42" x2="340.36" y2="185.42" width="0.1524" layer="91"/>
-<pinref part="RN2" gate="G$1" pin="8"/>
-</segment>
-</net>
-<net name="N$15" class="0">
-<segment>
-<pinref part="CON2" gate="G$1" pin="5"/>
-<wire x1="327.66" y1="182.88" x2="340.36" y2="182.88" width="0.1524" layer="91"/>
-<pinref part="RN2" gate="G$1" pin="7"/>
 </segment>
 </net>
@@
 <net name="N$19" class="0">
 <segment>
+<pinref part="RN2" gate="G$1" pin="5"/>
 <pinref part="CON2" gate="G$1" pin="6"/>
-<pinref part="RN2" gate="G$1" pin="5"/>
-<wire x1="330.2" y1="180.34" x2="340.36" y2="180.34" width="0.1524" layer="91"/>
-<wire x1="327.66" y1="177.8" x2="330.2" y2="177.8" width="0.1524" layer="91"/>
-<wire x1="330.2" y1="177.8" x2="330.2" y2="180.34" width="0.1524" layer="91"/>
+<wire x1="340.36" y1="180.34" x2="322.58" y2="180.34" width="0.1524" layer="91"/>
 </segment>
 </net>
 <net name="CLOCK_BUFFERED" class="0">
 <segment>
-<wire x1="314.96" y1="182.88" x2="312.42" y2="182.88" width="0.1524" layer="91"/>
-<label x="312.42" y="182.88" size="1.27" layer="95" rot="R180" xref="yes"/>
-<pinref part="RN2" gate="G$1" pin="2"/>
+<label x="304.8" y="180.34" size="1.27" layer="95" rot="R180" xref="yes"/>
+<pinref part="RN2" gate="G$1" pin="4"/>
+<wire x1="304.8" y1="180.34" x2="309.88" y2="180.34" width="0.1524" layer="91"/>
 </segment>
 <segment>
@@
 </segment>
 <segment>
-<wire x1="314.96" y1="185.42" x2="312.42" y2="185.42" width="0.1524" layer="91"/>
-<label x="312.42" y="185.42" size="1.27" layer="95" rot="R180" xref="yes"/>
-<pinref part="RN2" gate="G$1" pin="1"/>
+<label x="304.8" y="182.88" size="1.27" layer="95" rot="R180" xref="yes"/>
+<pinref part="RN2" gate="G$1" pin="3"/>
+<wire x1="304.8" y1="182.88" x2="309.88" y2="182.88" width="0.1524" layer="91"/>
 </segment>
 </net>
@@
 <net name="CS_OUT" class="0">
 <segment>
-<label x="309.88" y="177.8" size="1.27" layer="95" rot="R180" xref="yes"/>
-<pinref part="RN2" gate="G$1" pin="4"/>
-<wire x1="314.96" y1="177.8" x2="309.88" y2="177.8" width="0.1524" layer="91"/>
+<label x="297.18" y="187.96" size="1.27" layer="95" rot="R180" xref="yes"/>
+<pinref part="RN2" gate="G$1" pin="1"/>
+<wire x1="297.18" y1="187.96" x2="309.88" y2="187.96" width="0.1524" layer="91"/>
 </segment>
 <segment>
@@
 </segment>
 </net>
+<net name="N$7" class="0">
+<segment>
+<pinref part="CON2" gate="G$1" pin="5"/>
+<wire x1="322.58" y1="182.88" x2="340.36" y2="182.88" width="0.1524" layer="91"/>
+<pinref part="RN2" gate="G$1" pin="6"/>
+</segment>
+</net>
+<net name="N$8" class="0">
+<segment>
+<pinref part="RN2" gate="G$1" pin="8"/>
+<wire x1="322.58" y1="187.96" x2="327.66" y2="187.96" width="0.1524" layer="91"/>
+<wire x1="327.66" y1="187.96" x2="327.66" y2="185.42" width="0.1524" layer="91"/>
+<pinref part="CON2" gate="G$1" pin="4"/>
+<wire x1="327.66" y1="185.42" x2="340.36" y2="185.42" width="0.1524" layer="91"/>
+</segment>
+</net>

Commit message: PCB finalization
Parts:
- removed C27: 4.7u, rc:C-1206
- removed C28: 0.1u, rc:C-1206
- added C1, C2, C3, C4: 4.7 uF, rc:C-0603
- added C5: (no value), rc:C-1812
- added CON5, CON6, CON7: PINHEAD_1X01-2.54, pinhead:PINHEAD_1X01-2.54
- added PAD1, PAD2, PAD4: WIREPADSMD2.5-1.8, valenok_master_library:WIREPADSMD2.5-1.8
- added R1, R2: 100R, rc:R-0603
- added SJ4: (no value), eth_conv_master_lib:SOLDER_JOINT
- added TP1, TP2, TP3, TP4: PAD.05, pixhawk2:PAD.05
- added U$1: RTU, logo:RTU
- CON4: value PINHEAD_1X03-2.54 -> PINHEAD_1X01-2.54; device pinhead:PINHEAD_1X03-2.54 -> pinhead:PINHEAD_1X01-2.54
- IC8: device pixel_masterlib:LM317 -> masterlib:LM317
- LED_ANODE, LED_CATHODE1, LED_CATHODE2, LED_CATHODE3: device wirepad:WIREPADSMD5-2,5 -> valenok_master_library:WIREPADSMD5-2,5
- MODULE1: device pixel_masterlib:GW1584 -> ali_modules:GW1584
- R13: device rc:R-0805 -> rc:R-0603
- SJ1, SJ2, SJ3: device misc:SOLDER_JOINT -> eth_conv_master_lib:SOLDER_JOINT
- Z1: device crystals:CRYSTAL-3.2X2.5-4P -> watchdog_master_library:CRYSTAL-3.2X2.5-4P
Connections:
- removed net LED1: R39.2
- new net CURRENT_SENS: C3.2, R2.2, TP3.P$1
- new net LED_CATHODE: C1.1
- new net N$15: CON2.5, RN2.7
- new net STAT_LED: IC1.PA11, R39.2
- new net SUPPLY: C2.2, IC1.VCC
- new net SWCLK: IC1.PA14, PAD1.P, TP4.P$1
- new net SWIO: IC1.PA13, PAD2.P, TP1.P$1
- net CLOCK_BUFFERED: now also RN2.2; no longer RN2.4
- net CS_OUT: now also RN2.4; no longer RN2.1
- net DATA_BUFFERED: now also RN2.1; no longer RN2.3
- net GND: now also C1.1, C2.1, C3.1, C4.1, C5.1, PAD4.P, R2.1, R2.2, TP2.P$1, TP4.P$1; no longer C27.1, C28.1, CON4.2, LED2.C
- net GNDD: now also LED2.C
- net LED1_PWM: now also IC1.PA10/C3; no longer IC1.PA8/C1
- net LED2_CURRENT: now also IC1.PA6; no longer IC1.PB0/C2N
- net LED3_CURRENT: now also IC1.PA5; no longer IC1.PB1/C3N
- net LED3_PWM: now also IC1.PA8/C1; no longer IC1.PA10/C3
- net LED_ANODE: now also C1.2
- net N$10: now also CON5.1
- net N$2: now also C1.2, C2.2, C3.2, C4.2, IC8.OUT, R6.2, SJ4.2, TP2.P$1; no longer CON4.1, IC1.PA14
- net N$21: now also CON6.1
- net N$23: now also CON7.1
- net N$3: now also IC1.PB1/C3N, R1.1, R2.1; no longer CON4.3, IC1.PA13
- net N$5: now also C5.2; no longer C28.2
- net N$7: now also R1.2; no longer CON2.5, RN2.6
- net PWM: now also TP1.P$1
- net VDD_12V: no longer IC1.VCC
- net VDD_24V: now also CON4.1
- net VDD_3V3: now also R1.2, SJ4.1, TP3.P$1; no longer C27.2, IC8.OUT, R6.2
- net VIN_SENSE: now also IC1.PB0/C2N
Other:
- note added: "Do not use"
- note added: "R1, R2, R3 are for software version definition"
- note added: "SJ4 is for current consumption measurement"
- note removed: "STAT"
- moved on the sheet: C18, LED_ANODE, LED_CATHODE1, LED_CATHODE2, LED_CATHODE3, R10, R13, RN2

Commit message: PCB Finalization #2
Parts:
- added FRAME1: RTU_A4, frames:RTU_A4
- added FRAME2: RTU_A3, frames:RTU_A3
Connections:
- net LED1_CURRENT: now also IC1.PA6; no longer IC1.PA7/C1N
- net LED2_CURRENT: now also IC1.PA7/C1N; no longer IC1.PA6
- net LED3_CURRENT: now also IC1.PB0/C2N; no longer IC1.PA5
- net VIN_SENSE: now also IC1.PA5; no longer IC1.PB0/C2N
Other:
- moved on the sheet: C1, C2, C3, C4, C5, IC8, MODULE1, R6, R7, SJ1, SJ3, SJ4
