File: pixel8.sch (EAGLE design)
At the start: 18 parts, among them CON3 DS1066-07M-SIDE, CON4 DS1066-07M-SIDE

Commit message: pixel8 update
Parts:
- removed CON4: DS1066-07M-SIDE, pixel_masterlib:DS1066-07M-SIDE
- removed D1, D2, D3: (no value), SparkFun-DiscreteSemi:DIODESMA-KIT
- removed IC1, IC2, IC3: (no value), PT4115:PT4115
- removed L1, L2, L3: 68uH, inductor-panasonic:ELL6
- removed R3: 0.3, SparkFun-Resistors:0.3OHM-1/8W-1%(0805)
- added ANODE1, ANODE2, ANODE3, CATHODE1, CATHODE2, CATHODE3: WIREPADSMD5-2,5, valenok_master_library:WIREPADSMD5-2,5
- added C19, C20: (no value), rc:C-0603
- added C26: 100 nF, rc:C-0603
- added CON1, CON2: DS1066-07M-SIDE, pixel_masterlib:DS1066-07M-SIDE
- added D4: SMF05C, pixel_masterlib:SMF05C
- added IC4: ST3485SOIC8, pixel_masterlib:ST3485SOIC8
- added IC6, IC7: MC74VHC1GT125, pixel_masterlib:MC74VHC1GT125
- added R5: 120R, rc:R-0603
- added R8: 10K, rc:R-0603
- added RN1, RN2: 510R, pixel_masterlib:RESISTOR_ARRAY
- added SJ2: (no value), eth_conv_master_lib:SOLDER_JOINT
- added U$6: CONNECTION, usb2can_master_lib:CONNECTION
- added Z1: 16MHz, watchdog_master_library:CRYSTAL-3.2X2.5-4P
- C1: value 22uF -> 0.1uF; device rcl:CPOL-EUD/7343-31R -> rc:C-0603
- C2, C3: value 22uF -> 100 nF; device rcl:CPOL-EUD/7343-31R -> rc:C-0603
- CON3: value DS1066-07M-SIDE -> PINHEAD_1X02-2.54; device pixel_masterlib:DS1066-07M-SIDE -> pinhead:PINHEAD_1X02-2.54
- R1, R2: value 0.3 -> 100R; device SparkFun-Resistors:0.3OHM-1/8W-1%(0805) -> rc:R-0603
Connections:
- removed net B+: IC3.CSN, R3.1
- removed net B-: L3.1
- removed net G+: IC2.CSN, R2.1
- removed net G-: L2.1
- removed net N$14: CON3.4
- removed net N$16: CON3.5
- removed net N$18: CON3.6
- removed net N$19: CON4.4
- removed net N$20: CON4.5
- removed net N$21: CON4.6
- removed net PWM_B: IC3.DIM
- removed net PWM_G: IC2.DIM
- removed net PWM_R: IC1.DIM
- removed net R+: IC1.CSN, R1.1
- removed net R-: L1.1
- removed net RS485_A: CON3.2, CON4.2
- removed net RS485_B: CON3.3, CON4.3
- removed net VCC: C1.+, C2.+, C3.+, D1.C, D2.C, D3.C, IC1.VIN, IC2.VIN, IC3.VIN, R1.2, R2.2, R3.2
- removed net VDD_24V: CON3.1, CON4.1
- new net A: D4.D3, IC4.A, R2.1, R5.2
- new net ANODE: R1.1
- new net B: D4.D2, IC4.B, R1.1, SJ2.1
- new net CLOCK: D4.D5, IC6.IN_A, MODULE1.C5, RN1.3
- new net CLOCK_BUFFERED: IC6.OUT_Y, RN2.2
- new net CS: D4.D1, MODULE1.A3, RN1.4
- new net CS_OUT: MODULE1.C3, RN2.4
- new net DATA_BUFFERED: IC7.OUT_Y, RN2.1
- new net GNDD: CON1.7, CON2.7, U$6.P$1
- new net MISO: MODULE1.C7
- new net MOSI/DATA: D4.D4, IC7.IN_A, MODULE1.C6, RN1.2
- new net N$1: CON2.4, RN2.8
- new net N$10: ANODE1.P
- new net N$11: CON1.4, RN1.7
- new net N$12: CON1.5, RN1.6
- new net N$13: CON1.6, RN1.5
- new net N$15: CON2.5, RN2.7
- new net N$17: ANODE3.P
- new net N$3: CON2.6, RN2.5
- new net N$5: R5.1, SJ2.2
- new net N$6: C19.1, MODULE1.A1, Z1.1
- new net N$8: CATHODE1.P
- new net N$9: C20.1, MODULE1.A2, Z1.2
- new net PWM1: MODULE1.D4
- new net PWM2: MODULE1.D3
- new net PWM3: MODULE1.D2
- new net RE/DE: IC4.!RE, IC4.DE, MODULE1.D6
- new net RS485_A1: CON1.2, CON2.2, R1.2
- new net RS485_B1: CON1.3, CON2.3, R2.2
- new net RX/TX: IC4.DI, IC4.RO, MODULE1.D5
- new net SUPPLY: C1.2, R1.2
- new net SWIM: MODULE1.D1
- new net TEMP: C26.2, CON3.1, MODULE1.C4, R8.2
- new net VDD_12V: CON1.1, CON2.1
- new net VDD_3V3: C1.2, C2.2, C3.2, CON3.2, IC4.VCC, IC6.VCC, IC7.VCC, MODULE1.3V3
- net GND: now also C1.1, C19.2, C2.1, C20.2, C26.1, C3.1, D4.G, IC4.GND, IC6.GND, IC7.GND, MODULE1.GND, R8.1, U$6.P$2, Z1.GND; no longer C1.-, C2.-, C3.-, CON3.7, CON4.7, IC1.GND, IC2.GND, IC3.GND
- net N$2: now also CATHODE2.P; no longer D1.A, IC1.SW, L1.2
- net N$4: now also ANODE2.P; no longer D2.A, IC2.SW, L2.2
- net N$7: now also CATHODE3.P; no longer D3.A, IC3.SW, L3.2
Other:
- note added: "RS485"
- note added: "UART should be used in single wire half-duplex mode"
- moved on the sheet: MODULE1

Commit message: pixel8 update
Parts:
- renumbered C19 to C4, C20 to C5, C26 to C6, R8 to R3
Connections:
- net N$10 renamed A1
- net N$17 renamed A3
- net N$2 renamed C2
- net N$4 renamed A2
- net N$7 renamed C3
- net N$8 renamed C1
- net RS485_A1 renamed RS485_A
- net RS485_B1 renamed RS485_B
Changed lines of the file:
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@@
 </segment>
 </net>
-<net name="N$2" class="0">
+<net name="SW" class="0">
 <segment>
 <pinref part="D1" gate="G$1" pin="A"/>
@@
 <part name="CATHODE1" library="valenok_master_library" deviceset="WIREPAD" device="SMD5-2,5"/>
 <part name="ANODE1" library="valenok_master_library" deviceset="WIREPAD" device="SMD5-2,5"/>
-<part name="R8" library="rc" deviceset="R" device="-0603" value="10K"/>
+<part name="R3" library="rc" deviceset="R" device="-0603" value="10K"/>
 <part name="CON3" library="pinhead" deviceset="PINHEAD_1X02" device="-2.54"/>
 <part name="GND18" library="supply_symbols" deviceset="GND" device="" value="GND"/>
 <part name="+P15" library="supply_symbols" deviceset="3.3V" device=""/>
-<part name="C26" library="rc" deviceset="C" device="-0603" value="100 nF"/>
+<part name="C6" library="rc" deviceset="C" device="-0603" value="100 nF"/>
 <part name="GND32" library="supply_symbols" deviceset="GND" device="" value="GND"/>
 <part name="+P7" library="supply_symbols" deviceset="12V" device=""/>
@@
 <part name="GND22" library="supply_symbols" deviceset="GNDD" device="" value="GNDD"/>
 <part name="GND23" library="supply_symbols" deviceset="GNDD" device="" value="GNDD"/>
-<part name="C19" library="rc" deviceset="C" device="-0603"/>
-<part name="C20" library="rc" deviceset="C" device="-0603"/>
+<part name="C4" library="rc" deviceset="C" device="-0603"/>
+<part name="C5" library="rc" deviceset="C" device="-0603"/>
 <part name="GND20" library="supply_symbols" deviceset="GND" device="" value="GND"/>
 <part name="Z1" library="watchdog_master_library" deviceset="CRYSTAL" device="-3.2X2.5-4P" value="16MHz"/>
@@
 </plain>
 <moduleinsts>
-<moduleinst name="LED_DRV1" module="PT4115" x="223.52" y="160.02" smashed="yes">
-<attribute name="NAME" x="223.52" y="160.02" size="2.032" layer="95" align="bottom-center"/>
+<moduleinst name="LED_DRV1" module="PT4115" x="223.52" y="160.02" offset="100" smashed="yes">
+<attribute name="NAME" x="223.52" y="168.656" size="2.032" layer="95" align="bottom-center"/>
 </moduleinst>
-<moduleinst name="LED_DRV2" module="PT4115" x="223.52" y="132.08" smashed="yes">
-<attribute name="NAME" x="223.52" y="132.08" size="2.032" layer="95" align="bottom-center"/>
+<moduleinst name="LED_DRV2" module="PT4115" x="223.52" y="132.08" offset="200" smashed="yes">
+<attribute name="NAME" x="223.52" y="140.716" size="2.032" layer="95" align="bottom-center"/>
 </moduleinst>
-<moduleinst name="LED_DRV3" module="PT4115" x="223.52" y="104.14" smashed="yes">
-<attribute name="NAME" x="223.52" y="104.14" size="2.032" layer="95" align="bottom-center"/>
+<moduleinst name="LED_DRV3" module="PT4115" x="223.52" y="104.14" offset="300" smashed="yes">
+<attribute name="NAME" x="223.52" y="112.776" size="2.032" layer="95" align="bottom-center"/>
 </moduleinst>
 </moduleinsts>
@@
 <instance part="CATHODE1" gate="G$1" x="248.92" y="154.94" rot="R180"/>
 <instance part="ANODE1" gate="G$1" x="248.92" y="165.1" rot="R180"/>
-<instance part="R8" gate="G$1" x="93.98" y="88.9" rot="MR90"/>
+<instance part="R3" gate="G$1" x="93.98" y="88.9" rot="MR90"/>
 <instance part="CON3" gate="G$1" x="104.14" y="93.98" rot="MR0"/>
 <instance part="GND18" gate="1" x="93.98" y="78.74"/>
 <instance part="+P15" gate="G$1" x="93.98" y="101.6"/>
-<instance part="C26" gate="G$1" x="88.9" y="88.9" rot="R90"/>
+<instance part="C6" gate="G$1" x="88.9" y="88.9" rot="R90"/>
 <instance part="GND32" gate="1" x="88.9" y="78.74"/>
 <instance part="+P7" gate="G$1" x="238.76" y="83.82"/>
@@
 <instance part="GND22" gate="G$1" x="238.76" y="27.94" rot="MR0"/>
 <instance part="GND23" gate="G$1" x="238.76" y="60.96" rot="MR0"/>
-<instance part="C19" gate="G$1" x="20.32" y="101.6" rot="MR0"/>
-<instance part="C20" gate="G$1" x="20.32" y="91.44" rot="MR0"/>
+<instance part="C4" gate="G$1" x="20.32" y="101.6" rot="MR0"/>
+<instance part="C5" gate="G$1" x="20.32" y="91.44" rot="MR0"/>
 <instance part="GND20" gate="1" x="15.24" y="86.36"/>
 <instance part="Z1" gate="P" x="25.4" y="96.52" rot="R270"/>
@@
 <segment>
 <wire x1="88.9" y1="81.28" x2="88.9" y2="86.36" width="0.1524" layer="91"/>
-<pinref part="C26" gate="G$1" pin="1"/>
+<pinref part="C6" gate="G$1" pin="1"/>
 <pinref part="GND32" gate="1" pin="GND"/>
 </segment>
@@
 <wire x1="93.98" y1="81.28" x2="93.98" y2="83.82" width="0.1524" layer="91"/>
 <pinref part="GND18" gate="1" pin="GND"/>
-<pinref part="R8" gate="G$1" pin="1"/>
+<pinref part="R3" gate="G$1" pin="1"/>
 </segment>
 <segment>
@@
 <segment>
 <pinref part="GND20" gate="1" pin="GND"/>
-<pinref part="C20" gate="G$1" pin="2"/>
+<pinref part="C5" gate="G$1" pin="2"/>
 <wire x1="15.24" y1="101.6" x2="15.24" y2="96.52" width="0.1524" layer="91"/>
 <wire x1="15.24" y1="96.52" x2="15.24" y2="91.44" width="0.1524" layer="91"/>
@@
 <wire x1="15.24" y1="91.44" x2="15.24" y2="88.9" width="0.1524" layer="91"/>
 <junction x="15.24" y="91.44"/>
-<pinref part="C19" gate="G$1" pin="2"/>
+<pinref part="C4" gate="G$1" pin="2"/>
 <wire x1="17.78" y1="101.6" x2="15.24" y2="101.6" width="0.1524" layer="91"/>
 <pinref part="Z1" gate="P" pin="GND"/>
@@
 <junction x="93.98" y="96.52"/>
 <wire x1="88.9" y1="91.44" x2="88.9" y2="96.52" width="0.1524" layer="91"/>
-<pinref part="C26" gate="G$1" pin="2"/>
-<pinref part="R8" gate="G$1" pin="2"/>
+<pinref part="C6" gate="G$1" pin="2"/>
+<pinref part="R3" gate="G$1" pin="2"/>
 <pinref part="CON3" gate="G$1" pin="1"/>
 <pinref part="MODULE1" gate="G$1" pin="C4"/>
@@
 </segment>
 </net>
-<net name="RS485_B1" class="0">
+<net name="RS485_B" class="0">
 <segment>
 <pinref part="CON2" gate="G$1" pin="3"/>
@@
 </segment>
 </net>
-<net name="RS485_A1" class="0">
+<net name="RS485_A" class="0">
 <segment>
 <pinref part="CON2" gate="G$1" pin="2"/>
@@
 <net name="N$6" class="0">
 <segment>
-<pinref part="C19" gate="G$1" pin="1"/>
+<pinref part="C4" gate="G$1" pin="1"/>
 <pinref part="Z1" gate="P" pin="1"/>
 <wire x1="25.4" y1="101.6" x2="22.86" y2="101.6" width="0.1524" layer="91"/>
@@
 <net name="N$9" class="0">
 <segment>
-<pinref part="C20" gate="G$1" pin="1"/>
+<pinref part="C5" gate="G$1" pin="1"/>
 <pinref part="Z1" gate="P" pin="2"/>
 <wire x1="25.4" y1="91.44" x2="22.86" y2="91.44" width="0.1524" layer="91"/>
@@
 </segment>
 </net>
-<net name="N$8" class="0">
+<net name="C1" class="0">
 <segment>
 <pinref part="CATHODE1" gate="G$1" pin="P"/>
@@
 </segment>
 </net>
-<net name="N$10" class="0">
+<net name="A1" class="0">
 <segment>
 <pinref part="ANODE1" gate="G$1" pin="P"/>
@@
 </segment>
 </net>
-<net name="N$2" class="0">
+<net name="C2" class="0">
 <segment>
 <pinref part="CATHODE2" gate="G$1" pin="P"/>
@@
 </segment>
 </net>
-<net name="N$4" class="0">
+<net name="A2" class="0">
 <segment>
 <pinref part="ANODE2" gate="G$1" pin="P"/>
@@
 </segment>
 </net>
-<net name="N$7" class="0">
+<net name="C3" class="0">
 <segment>
 <pinref part="CATHODE3" gate="G$1" pin="P"/>
@@
 </segment>
 </net>
-<net name="N$17" class="0">
+<net name="A3" class="0">
 <segment>
 <pinref part="ANODE3" gate="G$1" pin="P"/>

Commit message: -blah
Parts:
- added CON15: (no value), led_matrix_master_lib:B2B-PH-K-S
Connections:
- new net VDD_24V: CON15.-
- net GND: now also CON15.+
Changed lines of the file:
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@@
 <part name="+P5" library="supply_symbols" deviceset="3.3V" device=""/>
 <part name="+P6" library="supply_symbols" deviceset="12V" device=""/>
+<part name="CON15" library="led_matrix_master_lib" deviceset="B2B-PH-K-S" device=""/>
+<part name="GND17" library="supply_symbols" deviceset="GND" device="" value="GND"/>
 </parts>
 <sheets>
@@
 <instance part="+P5" gate="G$1" x="38.1" y="91.44" rot="MR270"/>
 <instance part="+P6" gate="G$1" x="200.66" y="167.64"/>
+<instance part="CON15" gate="G$1" x="149.86" y="55.88" rot="R270"/>
+<instance part="GND17" gate="1" x="142.24" y="48.26"/>
 </instances>
 <busses>
@@
 <wire x1="33.02" y1="96.52" x2="33.02" y2="88.9" width="0.1524" layer="91"/>
 </segment>
+<segment>
+<pinref part="GND17" gate="1" pin="GND"/>
+<pinref part="CON15" gate="G$1" pin="+"/>
+<wire x1="144.78" y1="53.34" x2="142.24" y2="53.34" width="0.1524" layer="91"/>
+<wire x1="142.24" y1="53.34" x2="142.24" y2="50.8" width="0.1524" layer="91"/>
+</segment>
 </net>
 <net name="TEMP" class="0">
@@
 </segment>
 </net>
+<net name="VDD_24V" class="0">
+<segment>
+<pinref part="CON15" gate="G$1" pin="-"/>
+<wire x1="144.78" y1="55.88" x2="137.16" y2="55.88" width="0.1524" layer="91"/>
+</segment>
+</net>
