File: LE table/CONNECTOR.brd (EAGLE design)
At the start: 10 x 70 mm, 2 parts, among them CON1 CONNECTOR, CON3 CONNECTOR

Commit message: blah
Parts:
- added E$1, E$2: (no value), pinhead:1X09-PTH_2
Connections:
- net N$1: now also E$1.1, E$2.9
- net N$8: now also E$1.2, E$2.8
Routing:
- net N$1: track 66.6 -> 0.00 mm, vias 0 -> 7
- net N$8: track 43.9 -> 0.00 mm
- net S$1: track 33.8 -> 0.00 mm, vias 8 -> 0
- added copper zone on layer 1, net N$1
- added copper zone on layer 16, net N$1
- added copper zone on layer 1, net N$8
Changed lines of the file:
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@@
 <setting verticaltext="up"/>
 </settings>
-<grid distance="0.025" unitdist="mm" unit="mm" style="lines" multiple="1" display="no" altdistance="0.025" altunitdist="inch" altunit="inch"/>
+<grid distance="5" unitdist="mm" unit="mm" style="lines" multiple="1" display="no" altdistance="0.025" altunitdist="inch" altunit="inch"/>
 <layers>
-<layer number="1" name="Top" color="4" fill="1" visible="no" active="yes"/>
+<layer number="1" name="Top" color="4" fill="1" visible="yes" active="yes"/>
 <layer number="2" name="Route2" color="1" fill="3" visible="no" active="no"/>
 <layer number="3" name="Route3" color="4" fill="3" visible="no" active="no"/>
@@
 <layer number="19" name="Unrouted" color="6" fill="1" visible="yes" active="yes"/>
 <layer number="20" name="Dimension" color="15" fill="1" visible="yes" active="yes"/>
-<layer number="21" name="tPlace" color="7" fill="1" visible="no" active="yes"/>
+<layer number="21" name="tPlace" color="7" fill="1" visible="yes" active="yes"/>
 <layer number="22" name="bPlace" color="7" fill="1" visible="yes" active="yes"/>
-<layer number="23" name="tOrigins" color="15" fill="1" visible="no" active="yes"/>
+<layer number="23" name="tOrigins" color="15" fill="1" visible="yes" active="yes"/>
 <layer number="24" name="bOrigins" color="15" fill="1" visible="yes" active="yes"/>
-<layer number="25" name="tNames" color="7" fill="1" visible="no" active="yes"/>
+<layer number="25" name="tNames" color="7" fill="1" visible="yes" active="yes"/>
 <layer number="26" name="bNames" color="7" fill="1" visible="yes" active="yes"/>
 <layer number="27" name="tValues" color="7" fill="1" visible="yes" active="yes"/>
@@
 <layer number="49" name="Reference" color="7" fill="1" visible="yes" active="yes"/>
 <layer number="50" name="dxf" color="7" fill="1" visible="no" active="no"/>
-<layer number="51" name="tDocu" color="7" fill="1" visible="no" active="yes"/>
+<layer number="51" name="tDocu" color="7" fill="1" visible="yes" active="yes"/>
 <layer number="52" name="bDocu" color="7" fill="1" visible="yes" active="yes"/>
 <layer number="53" name="tGND_GNDA" color="7" fill="9" visible="no" active="no"/>
@@
 <layer number="220" name="220bmp" color="21" fill="1" visible="no" active="no"/>
 <layer number="221" name="221bmp" color="22" fill="1" visible="no" active="no"/>
+<layer number="222" name="222bmp" color="23" fill="1" visible="no" active="no"/>
 <layer number="223" name="223bmp" color="24" fill="1" visible="no" active="no"/>
 <layer number="224" name="224bmp" color="25" fill="1" visible="no" active="no"/>
@@
 </class>
 </classes>
-<designrules name="default">
+<designrules name="default *">
 <description language="de">&lt;b&gt;EAGLE Design Rules&lt;/b&gt;
 &lt;p&gt;
@@
 <param name="mdViaViaSameLayer" value="8mil"/>
 <param name="mnLayersViaInSmd" value="2"/>
-<param name="mdCopperDimension" value="40mil"/>
+<param name="mdCopperDimension" value="0.3mm"/>
 <param name="mdDrill" value="8mil"/>
 <param name="mdSmdStop" value="0mil"/>
@@
 <param name="mlMinCreamFrame" value="0mil"/>
 <param name="mlMaxCreamFrame" value="0mil"/>
-<param name="mlViaStopLimit" value="0mil"/>
+<param name="mlViaStopLimit" value="40mil"/>
 <param name="srRoundness" value="0"/>
 <param name="srMinRoundness" value="0mil"/>
@@
 <attribute name="BOM" value="EXCLUDE" x="1.55" y="10" size="2" layer="27" font="vector" ratio="15" rot="R90" display="off"/>
 </element>
+<element name="E$1" library="pinhead" package="1X09-PTH_2" value="" x="1.55" y="60" rot="R90"/>
+<element name="E$2" library="pinhead" package="1X09-PTH_2" value="" x="1.55" y="10" rot="R90"/>
 </elements>
 <signals>
@@
 <contactref element="CON1" pad="1"/>
 <contactref element="CON3" pad="9"/>
-<wire x1="1.55" y1="52" x2="1.55" y2="18" width="1.6" layer="1"/>
-<wire x1="1.55" y1="50.6" x2="1.55" y2="18" width="1.6" layer="16"/>
-<wire x1="1.55" y1="18" x2="1.55" y2="18" width="0" layer="19" extent="1-16"/>
+<polygon width="0.3" layer="1" thermals="no">
+<vertex x="2.65" y="17.35"/>
+<vertex x="2.65" y="52.65"/>
+<vertex x="0.425" y="52.65"/>
+<vertex x="0.45" y="17.35"/>
+</polygon>
+<polygon width="0.3" layer="16" thermals="no">
+<vertex x="0.425" y="17.35"/>
+<vertex x="0.425" y="52.65"/>
+<vertex x="2.65" y="52.65"/>
+<vertex x="2.625" y="17.35"/>
+</polygon>
+<contactref element="E$1" pad="1"/>
+<contactref element="E$2" pad="9"/>
+<via x="1.5" y="50.2" extent="1-16" drill="0.5" shape="square"/>
+<via x="1.5" y="45.2" extent="1-16" drill="0.5" shape="square"/>
+<via x="1.5" y="40.2" extent="1-16" drill="0.5" shape="square"/>
+<via x="1.5" y="35.2" extent="1-16" drill="0.5" shape="square"/>
+<via x="1.5" y="30.2" extent="1-16" drill="0.5" shape="square"/>
+<via x="1.5" y="25.2" extent="1-16" drill="0.5" shape="square"/>
+<via x="1.5" y="20.2" extent="1-16" drill="0.5" shape="square"/>
 </signal>
 <signal name="N$8">
 <contactref element="CON3" pad="8"/>
 <contactref element="CON1" pad="2"/>
-<wire x1="1.55" y1="54" x2="3.25" y2="54" width="1.6" layer="1"/>
-<wire x1="3.25" y1="54" x2="3.95" y2="53.3" width="1.6" layer="1"/>
-<wire x1="3.95" y1="53.3" x2="3.95" y2="16.7" width="1.6" layer="1"/>
-<wire x1="3.95" y1="16.7" x2="3.25" y2="16" width="1.6" layer="1"/>
-<wire x1="3.25" y1="16" x2="1.55" y2="16" width="1.6" layer="1"/>
-<via x="4.125" y="52.95" extent="1-16" drill="0.3" diameter="0.6"/>
-<via x="3.5" y="53.3" extent="1-16" drill="0.3" diameter="0.6"/>
-<via x="3.5" y="54.05" extent="1-16" drill="0.3" diameter="0.6"/>
-<via x="4.125" y="53.675" extent="1-16" drill="0.3" diameter="0.6"/>
-<wire x1="4.125" y1="52.95" x2="4.125" y2="53.675" width="0.3" layer="16"/>
-<via x="4.15" y="16.35" extent="1-16" drill="0.3" diameter="0.6"/>
-<via x="3.5" y="16" extent="1-16" drill="0.3" diameter="0.6"/>
-<via x="3.5" y="16.75" extent="1-16" drill="0.3" diameter="0.6"/>
-<via x="4.15" y="17.075" extent="1-16" drill="0.3" diameter="0.6"/>
-<wire x1="4.125" y1="52.95" x2="3.5" y2="52.95" width="0.3" layer="16"/>
-<wire x1="3.5" y1="52.95" x2="3.5" y2="53.3" width="0.3" layer="16"/>
 <polygon width="0.3" layer="16" thermals="no">
-<vertex x="4.625" y="15.31"/>
-<vertex x="3.3" y="15.31"/>
-<vertex x="3.3" y="54.325"/>
-<vertex x="4.625" y="54.325"/>
+<vertex x="6.53" y="15.35"/>
+<vertex x="0.45" y="15.35"/>
+<vertex x="0.45" y="16.65"/>
+<vertex x="3.4" y="16.65"/>
+<vertex x="3.4" y="53.35"/>
+<vertex x="0.5" y="53.35"/>
+<vertex x="0.5" y="54.65"/>
+<vertex x="6.53" y="54.65"/>
 </polygon>
-<wire x1="3.25" y1="16" x2="3.5" y2="16" width="0.3" layer="1"/>
+<contactref element="E$1" pad="2"/>
+<contactref element="E$2" pad="8"/>
+<polygon width="0.3" layer="1" thermals="no">
+<vertex x="4.625" y="15.35"/>
+<vertex x="0.45" y="15.35"/>
+<vertex x="0.45" y="16.65"/>
+<vertex x="3.4" y="16.65"/>
+<vertex x="3.4" y="53.35"/>
+<vertex x="0.5" y="53.35"/>
+<vertex x="0.5" y="54.65"/>
+<vertex x="4.625" y="54.65"/>
+</polygon>
+<via x="4.05" y="52.75" extent="1-16" drill="0.5" shape="square"/>
+<via x="4.05" y="47.75" extent="1-16" drill="0.5" shape="square"/>
+<via x="4.05" y="42.75" extent="1-16" drill="0.5" shape="square"/>
+<via x="4.05" y="37.75" extent="1-16" drill="0.5" shape="square"/>
+<via x="4.05" y="32.75" extent="1-16" drill="0.5" shape="square"/>
+<via x="4.05" y="27.75" extent="1-16" drill="0.5" shape="square"/>
+<via x="4.05" y="22.75" extent="1-16" drill="0.5" shape="square"/>
+<via x="4.05" y="17.75" extent="1-16" drill="0.5" shape="square"/>
 </signal>
 <signal name="N$16">
@@
 </signal>
 <signal name="S$1">
-<via x="1.2" y="50.55" extent="1-16" drill="0.3" diameter="0.6"/>
-<via x="1.9" y="50.55" extent="1-16" drill="0.3" diameter="0.6"/>
-<via x="1.2" y="49.85" extent="1-16" drill="0.3" diameter="0.6"/>
-<via x="1.9" y="49.85" extent="1-16" drill="0.3" diameter="0.6"/>
-<wire x1="1.2" y1="49.85" x2="1.2" y2="50.55" width="0.3" layer="16"/>
-<wire x1="1.2" y1="50.55" x2="1.9" y2="50.55" width="0.3" layer="16"/>
-<wire x1="1.9" y1="50.55" x2="1.9" y2="49.85" width="0.3" layer="16"/>
-<via x="1.2" y="20.25" extent="1-16" drill="0.3" diameter="0.6"/>
-<via x="1.9" y="20.25" extent="1-16" drill="0.3" diameter="0.6"/>
-<via x="1.2" y="19.55" extent="1-16" drill="0.3" diameter="0.6"/>
-<via x="1.9" y="19.55" extent="1-16" drill="0.3" diameter="0.6"/>
-<wire x1="1.2" y1="19.55" x2="1.2" y2="20.25" width="0.3" layer="16"/>
-<wire x1="1.2" y1="20.25" x2="1.9" y2="20.25" width="0.3" layer="16"/>
-<wire x1="1.9" y1="20.25" x2="1.9" y2="19.55" width="0.3" layer="16"/>
-<wire x1="1.2" y1="20.25" x2="1.2" y2="49.85" width="0.3" layer="16"/>
 </signal>
 </signals>
