File: LE table/le_table.brd (EAGLE design)
At the start: 200 x 20 mm, 50 parts, among them CON2 CONNECTOR, CON5 CONNECTOR, IC1 LM2902DT, IC2 CD4066, IC3 M74HCT74, Q1 PHOTOTRANSISTOR-3MM, Q2 PHOTOTRANSISTOR-0805, Q3 PHOTOTRANSISTOR-3MM, Q4 PHOTOTRANSISTOR-0805, Q5 PHOTOTRANSISTOR-3MM, Q6 PHOTOTRANSISTOR-0805, Q7 PHOTOTRANSISTOR-3MM, Q8 PHOTOTRANSISTOR-0805

Commit message: blah
Parts:
- added CON3, CON4: PINHEAD_1X09-2, pinhead:1X09-PTH_2
- added D1, D2, D3, D4: BAR43AFILM, pixel_masterlib:SOT23-3
- added Q9: IRLML2502-SOT23, watchdog_master_library:SOT23B-3
- added R6: 2K, rc:R0805
- added SJ2: (no value), DAS_mater_library:RES_0
- moved U$3 80.0 mm to (-79.0, -5.33)
- moved U$6 80.0 mm to (-80.0, -5.33)
- moved U$7 80.0 mm to (-81.0, -5.33)
Connections:
- new net N$1: Q9.1, R6.1
- new net N$16: D1.3, RN1.1
- new net N$17: D2.3, RN1.2
- new net N$18: D3.3, RN1.3
- new net N$21: D4.3, RN1.4
- new net N$23: LED10.K, LED11.C, LED12.K, LED13.C, LED14.K, LED15.C, LED16.K, LED9.C, Q9.3, SJ2.1
- net AMP1: now also D1.1; no longer RN1.1
- net AMP2: now also D2.1; no longer RN1.2
- net AMP3: now also D3.1; no longer RN1.3
- net AMP4: now also D4.1; no longer RN1.4
- net CLK: now also CON3.5, CON4.5
- net DATA_IN: now also CON4.6
- net DATA_OUT: now also CON3.6, R6.2
- net GND: now also Q9.2, SJ2.2; no longer LED10.K, LED11.C, LED12.K, LED13.C, LED14.K, LED15.C, LED16.K, LED9.C
- net GNDD: now also CON3.9, CON4.9
- net SENSOR1: now also CON3.1, CON4.1
- net SENSOR2: now also CON3.2, CON4.2
- net SENSOR3: now also CON3.3, CON4.3
- net SENSOR4: now also CON3.4, CON4.4
- net VDD_5V: now also CON3.8, CON4.8
- net WS_DATA_IN: now also CON4.7
- net WS_DATA_OUT: now also CON3.7
Routing:
- net N$23: track 0.00 -> 161.2 mm, vias 0 -> 2
- net VDD_5V: track 119.6 -> 111.7 mm
- net N$16: track 0.00 -> 7.44 mm
- net N$21: track 0.00 -> 7.42 mm
- net N$17: track 0.00 -> 5.10 mm
- net N$18: track 0.00 -> 5.10 mm
- net AMP1: track 55.2 -> 59.8 mm
- net GND: track 14.8 -> 10.8 mm, vias 64 -> 70
- net AMP2: track 60.0 -> 63.5 mm
- net N$1: track 0.00 -> 3.33 mm
- net AMP4: track 57.9 -> 60.7 mm
- net DATA_OUT: track 187.5 -> 189.4 mm
- net AMP3: track 65.4 -> 67.0 mm
- net SENS4: track 79.7 -> 78.4 mm
- net WS_DATA_IN: track 22.0 -> 22.6 mm
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
Commit message: Software import
Parts:
- R1, R2, R3, R4: value 2K -> 15-20K
- R10, R11, R12, R9: value 240R -> 150R
- R6: value 2K -> 150R
- RN2: value (none) -> 150R
Connections:
- net VDD_5V: now also IC3.1, IC3.4
Routing:
- net VDD_5V: track 111.7 -> 133.9 mm
- net CLK: track 207.9 -> 207.2 mm
