File: LE table/le_table.sch (EAGLE design)
At the start: 48 parts, among them CON2 CONNECTOR, CON5 CONNECTOR, IC1 LM2902DT, IC2 CD4066, IC3 M74HCT74, Q1 PHOTOTRANSISTOR-3MM, Q2 PHOTOTRANSISTOR-0805, Q3 PHOTOTRANSISTOR-3MM, Q4 PHOTOTRANSISTOR-0805, Q5 PHOTOTRANSISTOR-3MM, Q6 PHOTOTRANSISTOR-0805, Q7 PHOTOTRANSISTOR-3MM, Q8 PHOTOTRANSISTOR-0805

Commit message: blah
Parts:
- added CON3, CON4: PINHEAD_1X09-2, pinhead:PINHEAD_1X09-2
- added D1, D2, D3, D4: BAR43AFILM, pixel_masterlib:BAR43AFILM
- added Q9: IRLML2502-SOT23, watchdog_master_library:IRLML2502-SOT23
- added R6: 2K, rc:R-0805
- added SJ2: (no value), DAS_mater_library:SOLDER_JOINT
Connections:
- new net N$1: Q9.G, R6.1
- new net N$16: D1.C, RN1.1
- new net N$17: D2.C, RN1.2
- new net N$18: D3.C, RN1.3
- new net N$21: D4.C, RN1.4
- new net N$23: LED10.C, LED11.C, LED12.C, LED13.C, LED14.C, LED15.C, LED16.C, LED9.C, Q9.D, SJ2.1
- net AMP1: now also D1.A; no longer RN1.1
- net AMP2: now also D2.A; no longer RN1.2
- net AMP3: now also D3.A; no longer RN1.3
- net AMP4: now also D4.A; no longer RN1.4
- net CLK: now also CON3.5, CON4.5
- net DATA_IN: now also CON4.6
- net DATA_OUT: now also CON3.6, R6.2
- net GND: now also Q9.S, SJ2.2; no longer LED10.C, LED11.C, LED12.C, LED13.C, LED14.C, LED15.C, LED16.C, LED9.C
- net GNDD: now also CON3.9, CON4.9
- net SENSOR1: now also CON3.1, CON4.1
- net SENSOR2: now also CON3.2, CON4.2
- net SENSOR3: now also CON3.3, CON4.3
- net SENSOR4: now also CON3.4, CON4.4
- net VDD_5V: now also CON3.8, CON4.8
- net WS_DATA_IN: now also CON4.7
- net WS_DATA_OUT: now also CON3.7
Other:
- moved on the sheet: C1, C2, C3, C4, LED1, LED10, LED11, LED12, LED13, LED14, LED15, LED16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

Commit message: Software import
Parts:
- CON3, CON4: BOM (none) -> EXCLUDE
- D1, D2, D3, D4, RN1: ASSY (none) -> DNM
- R1, R2, R3, R4: value 2K -> 15-20K
- R10, R11, R12, R9: value 240R -> 150R
- R6: value 2K -> 150R
- RN2: value (none) -> 150R
Connections:
- net VDD_5V: now also IC3.1!CLR, IC3.1!PR
Other:
- note added: "Replace IR leds and phototransistors with 1206 ones"
